File: PCB/HackPad.kicad_pcb (KiCad board)
At the start: 2 copper layers, 83.5 x 83.5 mm, 49 parts, among them SW1 SW_Push, SW10 SW_Push, SW11 SW_Push, SW12 SW_Push, SW13 SW_Push, SW14 SW_Push, SW15 SW_Push, SW16 SW_Push, SW2 SW_Push, SW3 SW_Push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

Commit message: Added mounting holes for PCB
Parts:
- added H1: MountingHole, MountingHole:MountingHole_3.5mm, F.Cu at (105.9, 98.8)
- added H2: MountingHole, MountingHole:MountingHole_3.5mm, F.Cu at (27.4, 98.8)
- added H3: MountingHole, MountingHole:MountingHole_3.5mm, F.Cu at (105.9, 20.3)
- added H4: MountingHole, MountingHole:MountingHole_3.5mm, F.Cu at (27.4, 20.3)

Commit message: Added .drl files
Parts:
- removed H1, H2, H3, H4: MountingHole, MountingHole:MountingHole_3.5mm
